Commit message: ARTR

File: src/gazebo_bot/urdf/artag.xacro (robot description, xacro)
@@ -3,5 +3,5 @@
 <link name="artag">
         <collision name="collision_tag">
-                <origin xyz="3 3 0.4" rpy="1.707 1.707 0" />
+                <origin xyz="0.3 0 0.4" rpy="1.707 1.707 0" />
                 <geometry>
                          <box size="0.5 0.5 0.5" />
@@ -9,5 +9,5 @@
         </collision>
 	<visual name="tag_visual">
-                <origin xyz="3 3 0.4" rpy="1.707 1.707 0" />
+                <origin xyz="0.3 0 0.4" rpy="1.707 1.707 0" />
                 <geometry>
                         <mesh filename= "file:///home/blebot/ar_tag/src/gazebo_bot/world/ar_tag.dae"/>
@@ -16,5 +16,5 @@
         <inertial>
                 <mass value="1.0" />
-                <origin xyz="3 3 0.0001" rpy="1.707 1.707 0"/>
+                <origin xyz="0.3 0  0.0001" rpy="1.707 1.707 0"/>
                 <inertia ixx="0.0001" ixy="0.0" ixz="0.0"
                          iyy="0.0001" iyz="0.0"

Commit message: ARTR

File: src/gazebo_bot/urdf/artag.xacro (robot description, xacro)
@@ -3,5 +3,5 @@
 <link name="artag">
         <collision name="collision_tag">
-                <origin xyz="0.3 0 0.4" rpy="1.707 1.707 0" />
+                <origin xyz="0.8 0 0.4" rpy="1.707 1.707 0" />
                 <geometry>
                          <box size="0.5 0.5 0.5" />
@@ -9,5 +9,5 @@
         </collision>
 	<visual name="tag_visual">
-                <origin xyz="0.3 0 0.4" rpy="1.707 1.707 0" />
+                <origin xyz="0.8 0 0.4" rpy="1.707 1.707 0" />
                 <geometry>
                         <mesh filename= "file:///home/blebot/ar_tag/src/gazebo_bot/world/ar_tag.dae"/>
@@ -16,5 +16,5 @@
         <inertial>
                 <mass value="1.0" />
-                <origin xyz="0.3 0  0.0001" rpy="1.707 1.707 0"/>
+                <origin xyz="0.8 0  0.0001" rpy="1.707 1.707 0"/>
                 <inertia ixx="0.0001" ixy="0.0" ixz="0.0"
                          iyy="0.0001" iyz="0.0"

Commit message: Update artag.xacro

File: src/gazebo_bot/urdf/artag.xacro (robot description, xacro)
@@ -11,5 +11,5 @@
                 <origin xyz="0.8 0 0.4" rpy="1.707 1.707 0" />
                 <geometry>
-                        <mesh filename= "file:///home/blebot/ar_tag/src/gazebo_bot/world/ar_tag.dae"/>
+                        <mesh filename= "$(find gazebo_bot)/world/ar_tag.dae"/>
                 </geometry>
         </visual>

Commit message: ARTR

File: src/gazebo_bot/urdf/artag.xacro (robot description, xacro)
@@ -11,5 +11,5 @@
                 <origin xyz="0.8 0 0.4" rpy="1.707 1.707 0" />
                 <geometry>
-                        <mesh filename= "$(find gazebo_bot)/world/ar_tag.dae"/>
+			<mesh filename= "$(find gazebo_bot)/ar_tag_blender/AR_tag1/ar_tag.dae"/>
                 </geometry>
         </visual>
