Commit message: ARTR

File: src/gazebo_bot/urdf/rover.xacro (robot description, xacro)
@@ -168,10 +168,10 @@
 <!--JOINTS -->
 <joint name="camera_joint_1" type="fixed">
-        <origin xyz="0.45 0.125 0.3" rpy="0 0 0.86" />
+        <origin xyz="-0.45 0.125 0.3" rpy="0 0 3.1414" />
         <child link="camera_1" />
         <parent link="chassis" />
 </joint>
 <joint name="camera_joint_2" type="fixed">
-        <origin xyz="0.45 -0.125 0.3" rpy="0 0 -0.86" />
+        <origin xyz="-0.45 -0.125 0.3" rpy="0 0 3.1414" />
         <child link="camera_2" />
         <parent link="chassis" />

Commit message: ARTR

File: src/gazebo_bot/urdf/rover.xacro (robot description, xacro)
@@ -168,15 +168,15 @@
 <!--JOINTS -->
 <joint name="camera_joint_1" type="fixed">
-        <origin xyz="-0.45 0.125 0.3" rpy="0 0 3.1414" />
+        <origin xyz="-0.45 0.125 0.3" rpy="0 0 2.35605" />
         <child link="camera_1" />
         <parent link="chassis" />
 </joint>
 <joint name="camera_joint_2" type="fixed">
-        <origin xyz="-0.45 -0.125 0.3" rpy="0 0 3.1414" />
+        <origin xyz="-0.45 -0.125 0.3" rpy="0 0 3.92675" />
         <child link="camera_2" />
         <parent link="chassis" />
 </joint>
   <joint type="continuous" name="left_wheel_hinge">
-    <origin xyz="0.35 0.565 0" rpy="0 0 0"/>
+    <origin xyz="0.25 0.565 0" rpy="0 0 0"/>
     <child link="left_wheel"/>
     <parent link="chassis"/>
@@ -186,5 +186,5 @@
   </joint>
   <joint type="continuous" name="right_wheel_hinge">
-    <origin xyz="0.35 -0.565 0" rpy="0 0 0"/>
+    <origin xyz="0.25 -0.565 0" rpy="0 0 0"/>
     <child link="right_wheel"/>
     <parent link="chassis"/>
@@ -194,5 +194,5 @@
   </joint>
  <joint type="continuous" name="left_wheel_fhinge">
-    <origin xyz="-0.35 0.565 0" rpy="0 0 0"/>
+    <origin xyz="-0.25 0.565 0" rpy="0 0 0"/>
     <child link="left_fwheel"/>
     <parent link="chassis"/>
@@ -202,5 +202,5 @@
   </joint>
   <joint type="continuous" name="right_wheel_fhinge">
-    <origin xyz="-0.35 -0.565 0" rpy="0 0 0"/>
+    <origin xyz="-0.25 -0.565 0" rpy="0 0 0"/>
     <child link="right_fwheel"/>
     <parent link="chassis"/>

Commit message: ARTR

File: src/gazebo_bot/urdf/rover.xacro (robot description, xacro)
@@ -32,4 +32,25 @@
         </collision>
         <visual name="camera_visual_2">
+                <origin xyz="0 0 0" rpy="0 0 0" />
+                <geometry>
+                        <box size="0.1 0.1 0.1" />
+                </geometry>
+        </visual>
+        <inertial>
+                <mass value="0.1" />
+                <origin xyz="0 0 0.0001" rpy="0 0 0"/>
+                <inertia ixx="0.0001" ixy="0.0" ixz="0.0"
+                         iyy="0.0001" iyz="0.0"
+                         izz="0.0001" />
+        </inertial>
+</link>
+<link name="lidar">
+        <collision name="collision_lidar">
+                <origin xyz="0 0 0" rpy="0 0 0" />
+                <geometry>
+                         <box size="0.1 0.1 0.1" />
+                </geometry>
+        </collision>
+        <visual name="camera_lidar">
                 <origin xyz="0 0 0" rpy="0 0 0" />
                 <geometry>
@@ -177,4 +198,9 @@
         <parent link="chassis" />
 </joint>
+<joint name="lidar_joint" type="fixed">
+        <origin xyz="-0.45 0 0.1" rpy="0 0 3.1414" />
+        <child link="lidar" />
+        <parent link="chassis" />
+</joint>
   <joint type="continuous" name="left_wheel_hinge">
     <origin xyz="0.25 0.565 0" rpy="0 0 0"/>

Commit message: .

File: src/gazebo_bot/urdf/rover.xacro (robot description, xacro)
@@ -1,8 +1,8 @@
 <?xml version='1.0'?>
 <robot name="rover" xmlns:xacro="http://www.ros.org/wiki/xacro">
-<xacro:include filename="/$(find gazebo_bot)/urdf/rover.gazebo" />
+<xacro:include filename="$(find gazebo_bot)/urdf/rover.gazebo" />
 <!-- CAMERAS-->
-<link name="camera_1">
-        <collision name="collision_camera_1">
+<link name="camera">
+        <collision name="collision_camera">
                 <origin xyz="0 0 0" rpy="0 0 0" />
                 <geometry>
@@ -10,5 +10,5 @@
                 </geometry>
         </collision>
-        <visual name="camera_visual_1">
+        <visual name="camera_visual">
                 <origin xyz="0 0 0" rpy="0 0 0" />
                 <geometry>
@@ -24,45 +24,22 @@
         </inertial>
 </link>
-<link name="camera_2">
-        <collision name="collision_camera_2">
-                <origin xyz="0 0 0" rpy="0 0 0" />
-                <geometry>
-                         <box size="0.1 0.1 0.1" />
-                </geometry>
-        </collision>
-        <visual name="camera_visual_2">
-                <origin xyz="0 0 0" rpy="0 0 0" />
-                <geometry>
-                        <box size="0.1 0.1 0.1" />
-                </geometry>
-        </visual>
-        <inertial>
-                <mass value="0.1" />
-                <origin xyz="0 0 0.0001" rpy="0 0 0"/>
-                <inertia ixx="0.0001" ixy="0.0" ixz="0.0"
-                         iyy="0.0001" iyz="0.0"
-                         izz="0.0001" />
-        </inertial>
-</link>
-<link name="lidar">
-        <collision name="collision_lidar">
-                <origin xyz="0 0 0" rpy="0 0 0" />
-                <geometry>
-                         <box size="0.1 0.1 0.1" />
-                </geometry>
-        </collision>
-        <visual name="camera_lidar">
-                <origin xyz="0 0 0" rpy="0 0 0" />
-                <geometry>
-                        <box size="0.1 0.1 0.1" />
-                </geometry>
-        </visual>
-        <inertial>
-                <mass value="0.1" />
-                <origin xyz="0 0 0.0001" rpy="0 0 0"/>
-                <inertia ixx="0.0001" ixy="0.0" ixz="0.0"
-                         iyy="0.0001" iyz="0.0"
-                         izz="0.0001" />
-        </inertial>
+<link name="hokuyo">
+    <collision>
+      <origin xyz="0 0 0" rpy="0 0 0"/>
+      <geometry>
+         <box size="0.1 0.1 0.1"/>
+      </geometry>
+    </collision>
+    <visual>
+      <origin xyz="0 0 0" rpy="0 0 0"/>
+      <geometry>
+        <mesh filename="package://gazebo_bot/meshes/hokuyo.dae"/>
+      </geometry>
+    </visual>
+    <inertial>
+      <mass value="1e-5" />
+      <origin xyz="0 0 0" rpy="0 0 0"/>
+      <inertia ixx="1e-6" ixy="0" ixz="0" iyy="1e-6" iyz="0" izz="1e-6" />
+    </inertial>
 </link>
 <!-- CHASSIS -->
@@ -188,17 +165,12 @@
   </link>
 <!--JOINTS -->
-<joint name="camera_joint_1" type="fixed">
-        <origin xyz="-0.45 0.125 0.3" rpy="0 0 2.35605" />
-        <child link="camera_1" />
+<joint name="camera_joint" type="fixed">
+        <origin xyz="-0.45 0 0.3" rpy="0 0 3.1414" />
+        <child link="camera" />
         <parent link="chassis" />
 </joint>
-<joint name="camera_joint_2" type="fixed">
-        <origin xyz="-0.45 -0.125 0.3" rpy="0 0 3.92675" />
-        <child link="camera_2" />
-        <parent link="chassis" />
-</joint>
-<joint name="lidar_joint" type="fixed">
-        <origin xyz="-0.45 0 0.1" rpy="0 0 3.1414" />
-        <child link="lidar" />
+<joint name="hokuyo_joint" type="fixed">
+        <origin xyz="-0.45 0 0.25" rpy="0 0 3.1414" />
+        <child link="hokuyo" />
         <parent link="chassis" />
 </joint>

Commit message: realsense

File: src/gazebo_bot/urdf/rover.xacro (robot description, xacro)
@@ -1,7 +1,30 @@
 <?xml version='1.0'?>
-<robot name="rover" xmlns:xacro="http://www.ros.org/wiki/xacro">
+<robot name="mybot" xmlns:xacro="http://www.ros.org/wiki/xacro">
 <xacro:include filename="$(find gazebo_bot)/urdf/rover.gazebo" />
-<!-- CAMERAS-->
-<link name="camera">
+<xacro:include filename="$(find realsense2_description)/urdf/_d435.urdf.xacro"/>
+  <link name="chassis">
+    <pose>0 0 0.1 0 0 0</pose>
+    <inertial>
+      <mass value="10.0"/>
+      <origin xyz="0.0 0 0.1" rpy=" 0 0 0"/>
+      <inertia
+          ixx="2.4" ixy="0" ixz="0"
+          iyy="2.4" iyz="0"
+          izz="2.4"
+      />
+    </inertial>
+    <collision name='collision'>
+      <geometry>
+        <box size="1.0 1.0 .1"/>
+      </geometry>
+    </collision>
+    <visual name='chassis_visual'>
+      <origin xyz="0 0 0" rpy=" 0 0 0"/>
+      <geometry>
+        <box size="1.0 1.0 .1"/>
+      </geometry>
+    </visual>
+  </link>
+<!--link name="camera">
         <collision name="collision_camera">
                 <origin xyz="0 0 0" rpy="0 0 0" />
@@ -23,5 +46,5 @@
                          izz="0.0001" />
         </inertial>
-</link>
+</link-->
 <link name="hokuyo">
     <collision>
@@ -43,31 +66,5 @@
     </inertial>
 </link>
-<!-- CHASSIS -->
-  <link name="chassis">
-    <pose>0 0 0.1 0 0 0</pose>
-    <inertial>
-      <mass value="10.0"/>
-      <origin xyz="0.0 0 0.1" rpy=" 0 0 0"/>
-      <inertia
-          ixx="2.4" ixy="0" ixz="0"
-          iyy="2.4" iyz="0"
-          izz="2.4"
-      />
-    </inertial>
-    <collision name='collision'>
-      <geometry>
-        <box size="1 1 .1"/>
-      </geometry>
-    </collision>
-    <visual name='chassis_visual'>
-      <origin xyz="0 0 0" rpy=" 0 0 0"/>
-      <geometry>
-        <box size="1 1 .1"/>
-      </geometry>
-    </visual>
-  </link>
-<!-- WHEEL LINKS -->
   <link name="left_wheel">
-    <!--origin xyz="0.1 0.13 0.1" rpy="0 1.5707 1.5707"-->
     <collision name="collision">
       <origin xyz="0 0 0" rpy="0 1.5707 1.5707"/>
@@ -93,5 +90,4 @@
   </link>
   <link name="right_wheel">
-    <!--origin xyz="0.1 -0.13 0.1" rpy="0 1.5707 1.5707"/-->
     <collision name="collision">
       <origin xyz="0 0 0" rpy="0 1.5707 1.5707"/>
@@ -117,5 +113,4 @@
   </link>
   <link name="left_fwheel">
-    <!--origin xyz="-0.1 0.13 0.1" rpy="0 1.5707 1.5707"-->
     <collision name="collision">
       <origin xyz="0 0 0" rpy="0 1.5707 1.5707"/>
@@ -141,5 +136,4 @@
   </link>
   <link name="right_fwheel">
-    <!--origin xyz="-0.1 -0.13 0.1" rpy="0 1.5707 1.5707"/-->
     <collision name="collision">
       <origin xyz="0 0 0" rpy="0 1.5707 1.5707"/>
@@ -164,47 +158,43 @@
     </inertial>
   </link>
-<!--JOINTS -->
-<joint name="camera_joint" type="fixed">
-        <origin xyz="-0.45 0 0.3" rpy="0 0 3.1414" />
-        <child link="camera" />
-        <parent link="chassis" />
-</joint>
+  <joint type="continuous" name="left_wheel_hinge">
+    <origin xyz="0.25 0.565 0" rpy="0 0 0"/>
+    <child link="left_wheel"/>
+    <parent link="chassis"/>
+    <axis xyz="0 1 0" rpy="0 0 0"/>
+    <limit effort="100" velocity="100"/>
+    <joint_properties damping="0.0" friction="1.0"/>
+  </joint>
+  <joint type="continuous" name="right_wheel_hinge">
+    <origin xyz="0.25 -0.565 0" rpy="0 0 0"/>
+    <child link="right_wheel"/>
+    <parent link="chassis"/>
+    <axis xyz="0 1 0" rpy="0 0 0"/>
+    <limit effort="100" velocity="100"/>
+    <joint_properties damping="0.0" friction="1.0"/>
+  </joint>
+ <joint type="continuous" name="left_wheel_fhinge">
+    <origin xyz="-0.25 0.565 0" rpy="0 0 0"/>
+    <child link="left_fwheel"/>
+    <parent link="chassis"/>
+    <axis xyz="0 1 0" rpy="0 0 0"/>
+    <limit effort="100" velocity="100"/>
+    <joint_properties damping="0.0" friction="1.0"/>
+  </joint>
+  <joint type="continuous" name="right_wheel_fhinge">
+    <origin xyz="-0.25 -0.565 0" rpy="0 0 0"/>
+    <child link="right_fwheel"/>
+    <parent link="chassis"/>
+    <axis xyz="0 1 0" rpy="0 0 0"/>
+    <limit effort="100" velocity="100"/>
+    <joint_properties damping="0.0" friction="1"/>
+  </joint>
 <joint name="hokuyo_joint" type="fixed">
-        <origin xyz="-0.45 0 0.25" rpy="0 0 3.1414" />
+        <origin xyz="0.45 0 0.25" rpy="0 0 0" />
         <child link="hokuyo" />
         <parent link="chassis" />
 </joint>
-  <joint type="continuous" name="left_wheel_hinge">
-    <origin xyz="0.25 0.565 0" rpy="0 0 0"/>
-    <child link="left_wheel"/>
-    <parent link="chassis"/>
-    <axis xyz="0 1 0" rpy="0 0 0"/>
-    <limit effort="100" velocity="100"/>
-    <joint_properties damping="0.0" friction="1.0"/>
-  </joint>
-  <joint type="continuous" name="right_wheel_hinge">
-    <origin xyz="0.25 -0.565 0" rpy="0 0 0"/>
-    <child link="right_wheel"/>
-    <parent link="chassis"/>
-    <axis xyz="0 1 0" rpy="0 0 0"/>
-    <limit effort="100" velocity="100"/>
-    <joint_properties damping="0.0" friction="1.0"/>
-  </joint>
- <joint type="continuous" name="left_wheel_fhinge">
-    <origin xyz="-0.25 0.565 0" rpy="0 0 0"/>
-    <child link="left_fwheel"/>
-    <parent link="chassis"/>
-    <axis xyz="0 1 0" rpy="0 0 0"/>
-    <limit effort="100" velocity="100"/>
-    <joint_properties damping="0.0" friction="1.0"/>
-  </joint>
-  <joint type="continuous" name="right_wheel_fhinge">
-    <origin xyz="-0.25 -0.565 0" rpy="0 0 0"/>
-    <child link="right_fwheel"/>
-    <parent link="chassis"/>
-    <axis xyz="0 1 0" rpy="0 0 0"/>
-    <limit effort="100" velocity="100"/>
-    <joint_properties damping="0.0" friction="1"/>
-  </joint>
-<!-- END -->
+<sensor_d435 parent="chassis" name="camera" >
+        <origin xyz="0.45 0 0.3" rpy="0 0 0" />
+</sensor_d435>
 </robot>
